File: yuzu-pcb.kicad_pcb (KiCad board)
At the start: 2 copper layers, 37 x 23 mm, 28 parts, among them J1 Conn_ARM_JTAG_SWD_10, J2 Conn_01x04, SW1 SW_SPST, U1 E73-2G4M08S1C, U2 SHT45, X2 32.768Khz

Commit message: Sent for production
Parts:
- turned SW1 to 0 degrees
Connections:
- SW1 pad 2: /RESET -> GND
- SW1 pad 3: GND -> /RESET
Routing:
- net /RESET: track 23.7 -> 26.0 mm
Changed lines of the file:
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@@
 		)
 	)
-	(property "REV" "A")
+	(property "REV" "B")
 	(net 0 "")
 	(net 1 "unconnected-(U1-P0.24-Pad35)")
@@
 	(footprint "yuzu:RKB2SJG250SMTRLFS"
 		(layer "F.Cu")
-		(at 128.74 103.1 180)
+		(at 128.74 103.1)
 		(descr "RKB2SJG250SMTR LFS-2")
 		(tags "Switch")
 		(property "Reference" "SW1"
-			(at 3.75 0 90)
+			(at -4.74 -0.35 -90)
 			(unlocked yes)
 			(layer "F.SilkS")
@@
 		)
 		(property "Value" "SW_SPST"
-			(at 0 0 180)
+			(at 0 0 360)
 			(layer "F.SilkS")
 			(hide yes)
@@
 		)
 		(property "Footprint" "yuzu:RKB2SJG250SMTRLFS"
-			(at 0 0 180)
+			(at 0 0 0)
 			(unlocked yes)
 			(layer "F.Fab")
@@
 		)
 		(property "Datasheet" ""
-			(at 0 0 180)
+			(at 0 0 0)
 			(unlocked yes)
 			(layer "F.Fab")
@@
 		)
 		(property "Description" "Double Pole Single Throw (DPST) Switch"
-			(at 0 0 180)
+			(at 0 0 0)
 			(unlocked yes)
 			(layer "F.Fab")
@@
 		)
 		(property "LCSC" "C2927788"
-			(at 0 0 180)
+			(at 0 0 0)
 			(unlocked yes)
 			(layer "F.Fab")
@@
 		(attr smd)
 		(fp_line
-			(start 2.1 0.4)
-			(end 2.1 -0.4)
+			(start -3.3 -1.075)
+			(end -3.3 -1.075)
 			(stroke
-				(width 0.2)
+				(width 0.1)
 				(type solid)
 			)
@@
 		)
 		(fp_line
-			(start -1.4 1.6)
-			(end 1.4 1.6)
+			(start -3.2 -1.075)
+			(end -3.2 -1.075)
+			(stroke
+				(width 0.1)
+				(type solid)
+			)
+			(layer "F.SilkS")
+		)
+		(fp_line
+			(start -2.1 -0.4)
+			(end -2.1 0.4)
 			(stroke
 				(width 0.2)
@@
 		)
 		(fp_line
-			(start -2.1 -0.4)
-			(end -2.1 0.4)
+			(start -1.4 1.6)
+			(end 1.4 1.6)
 			(stroke
 				(width 0.2)
@@
 		)
 		(fp_line
-			(start -3.2 -1.075)
-			(end -3.2 -1.075)
+			(start 2.1 0.4)
+			(end 2.1 -0.4)
 			(stroke
-				(width 0.1)
+				(width 0.2)
 				(type solid)
 			)
 			(layer "F.SilkS")
 		)
-		(fp_line
+		(fp_arc
 			(start -3.3 -1.075)
-			(end -3.3 -1.075)
+			(mid -3.25 -1.125)
+			(end -3.2 -1.075)
 			(stroke
 				(width 0.1)
@@
 			(layer "F.SilkS")
 		)
-		(fp_arc
-			(start -3.3 -1.075)
-			(mid -3.25 -1.125)
-			(end -3.2 -1.075)
+		(fp_line
+			(start -3.75 -2.6)
+			(end 3.75 -2.6)
 			(stroke
 				(width 0.1)
 				(type solid)
 			)
-			(layer "F.SilkS")
+			(layer "F.CrtYd")
 		)
 		(fp_line
-			(start 3.75 2.6)
-			(end -3.75 2.6)
+			(start -3.75 2.6)
+			(end -3.75 -2.6)
 			(stroke
 				(width 0.1)
@@
 		)
 		(fp_line
-			(start -3.75 2.6)
-			(end -3.75 -2.6)
+			(start 3.75 2.6)
+			(end -3.75 2.6)
 			(stroke
 				(width 0.1)
@@
 		)
 		(fp_line
-			(start -3.75 -2.6)
-			(end 3.75 -2.6)
+			(start -2.1 -1.6)
+			(end -2.1 1.6)
 			(stroke
 				(width 0.1)
 				(type solid)
 			)
-			(layer "F.CrtYd")
+			(layer "F.Fab")
 		)
 		(fp_line
-			(start 2.1 1.6)
-			(end 2.1 -1.6)
+			(start -2.1 1.6)
+			(end 2.1 1.6)
 			(stroke
 				(width 0.1)
@@
 		)
 		(fp_line
-			(start -2.1 1.6)
-			(end 2.1 1.6)
-			(stroke
-				(width 0.1)
-				(type solid)
-			)
-			(layer "F.Fab")
-		)
-		(fp_line
-			(start -2.1 -1.6)
-			(end -2.1 1.6)
+			(start 2.1 1.6)
+			(end 2.1 -1.6)
 			(stroke
 				(width 0.1)
@@
 		)
 		(fp_text user "${REFERENCE}"
-			(at 0 0 180)
+			(at 0 0 360)
 			(layer "F.Fab")
 			(effects
@@
 		)
 		(pad "1" smd rect
-			(at -2.25 -1.075 270)
+			(at -2.25 -1.075 90)
 			(size 0.7 1)
 			(layers "F.Cu" "F.Paste" "F.Mask")
@@
 		)
 		(pad "2" smd rect
-			(at 2.25 -1.075 270)
+			(at 2.25 -1.075 90)
 			(size 0.7 1)
 			(layers "F.Cu" "F.Paste" "F.Mask")
-			(net 33 "/RESET")
+			(net 24 "GND")
 			(pinfunction "2")
 			(pintype "passive")
 		)
 		(pad "3" smd rect
-			(at -2.25 1.075 270)
+			(at -2.25 1.075 90)
 			(size 0.7 1)
 			(layers "F.Cu" "F.Paste" "F.Mask")
-			(net 24 "GND")
+			(net 33 "/RESET")
 			(pinfunction "3")
 			(pintype "passive")
 		)
 		(pad "4" smd rect
-			(at 2.25 1.075 270)
+			(at 2.25 1.075 90)
 			(size 0.7 1)
 			(layers "F.Cu" "F.Paste" "F.Mask")
@@
 	)
 	(segment
+		(start 126.49 104.175)
+		(end 130.99 104.175)
+		(width 0.2)
+		(layer "F.Cu")
+		(net 33)
+	)
+	(segment
 		(start 115.39 105.51)
 		(end 115.38 105.5)
@@
 		(width 0.2)
 		(layer "F.Cu")
-		(net 33)
-	)
-	(segment
-		(start 126.49 104.175)
-		(end 126.49 102.025)
-		(width 0.2)
-		(layer "F.Cu")
