File: yuzu-pcb.kicad_sch (KiCad schematic)
At the start: 12 parts, among them J1 Conn_ARM_JTAG_SWD_10, SW1 SW_SPST, U1 E73-2G4M08S1C, U2 SHT45, X2 32.768Khz

Commit message: Update project
Parts:
- C1, C3: footprint Capacitor_SMD:C_0402_1005Metric_Pad0.74x0.62mm_HandSolder -> Capacitor_SMD:C_0402_1005Metric
- U1: footprint yuzu:E73-2G4M08S1C-52840_SMD -> yuzu:E73(2G4M08S1C) JLCPCB
Changed lines of the file:
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@@
 		)
 		(instances
-			(project "Yuzu"
+			(project "yuzu-pcb"
 				(path "/170d21ec-bdb4-4292-838e-4735dd755299"
 					(reference "J1")
@@
 		)
 		(instances
-			(project "Yuzu"
+			(project "yuzu-pcb"
 				(path "/170d21ec-bdb4-4292-838e-4735dd755299"
 					(reference "#FLG02")
@@
 		)
 		(instances
-			(project "Yuzu"
+			(project "yuzu-pcb"
 				(path "/170d21ec-bdb4-4292-838e-4735dd755299"
 					(reference "BT1")
@@
 		)
 		(instances
-			(project "Yuzu"
+			(project "yuzu-pcb"
 				(path "/170d21ec-bdb4-4292-838e-4735dd755299"
 					(reference "#PWR08")
@@
 		)
 		(instances
-			(project "Yuzu"
+			(project "yuzu-pcb"
 				(path "/170d21ec-bdb4-4292-838e-4735dd755299"
 					(reference "#PWR05")
@@
 		)
 		(instances
-			(project "Yuzu"
+			(project "yuzu-pcb"
 				(path "/170d21ec-bdb4-4292-838e-4735dd755299"
 					(reference "#PWR03")
@@
 		)
 		(instances
-			(project "Yuzu"
+			(project "yuzu-pcb"
 				(path "/170d21ec-bdb4-4292-838e-4735dd755299"
 					(reference "#PWR09")
@@
 		)
 		(instances
-			(project "Yuzu"
+			(project "yuzu-pcb"
 				(path "/170d21ec-bdb4-4292-838e-4735dd755299"
 					(reference "#FLG03")
@@
 		)
 		(instances
-			(project "Yuzu"
+			(project "yuzu-pcb"
 				(path "/170d21ec-bdb4-4292-838e-4735dd755299"
 					(reference "R2")
@@
 		)
 		(instances
-			(project "Yuzu"
+			(project "yuzu-pcb"
 				(path "/170d21ec-bdb4-4292-838e-4735dd755299"
 					(reference "#PWR01")
@@
 		)
 		(instances
-			(project "Yuzu"
+			(project "yuzu-pcb"
 				(path "/170d21ec-bdb4-4292-838e-4735dd755299"
 					(reference "R1")
@@
 		)
 		(instances
-			(project "Yuzu"
+			(project "yuzu-pcb"
 				(path "/170d21ec-bdb4-4292-838e-4735dd755299"
 					(reference "D1")
@@
 		)
 		(instances
-			(project "Yuzu"
+			(project "yuzu-pcb"
 				(path "/170d21ec-bdb4-4292-838e-4735dd755299"
 					(reference "#FLG05")
@@
 		)
 		(instances
-			(project "Yuzu"
+			(project "yuzu-pcb"
 				(path "/170d21ec-bdb4-4292-838e-4735dd755299"
 					(reference "#PWR07")
@@
 		)
 		(instances
-			(project "Yuzu"
+			(project "yuzu-pcb"
 				(path "/170d21ec-bdb4-4292-838e-4735dd755299"
 					(reference "#PWR04")
@@
 		)
 		(instances
-			(project "Yuzu"
+			(project "yuzu-pcb"
 				(path "/170d21ec-bdb4-4292-838e-4735dd755299"
 					(reference "#PWR010")
@@
 		)
 		(instances
-			(project "Yuzu"
+			(project "yuzu-pcb"
 				(path "/170d21ec-bdb4-4292-838e-4735dd755299"
 					(reference "X2")
@@
 		)
 		(instances
-			(project "Yuzu"
+			(project "yuzu-pcb"
 				(path "/170d21ec-bdb4-4292-838e-4735dd755299"
 					(reference "U2")
@@
 		)
 		(instances
-			(project "Yuzu"
+			(project "yuzu-pcb"
 				(path "/170d21ec-bdb4-4292-838e-4735dd755299"
 					(reference "#PWR02")
@@
 		)
 		(instances
-			(project "Yuzu"
+			(project "yuzu-pcb"
 				(path "/170d21ec-bdb4-4292-838e-4735dd755299"
 					(reference "R3")
@@
 		)
 		(instances
-			(project "Yuzu"
+			(project "yuzu-pcb"
 				(path "/170d21ec-bdb4-4292-838e-4735dd755299"
 					(reference "SW1")
@@
 			)
 		)
-		(property "Footprint" "Capacitor_SMD:C_0402_1005Metric_Pad0.74x0.62mm_HandSolder"
+		(property "Footprint" "Capacitor_SMD:C_0402_1005Metric"
 			(at 30.48 119.0752 0)
 			(effects
@@
 		)
 		(instances
-			(project "Yuzu"
+			(project "yuzu-pcb"
 				(path "/170d21ec-bdb4-4292-838e-4735dd755299"
 					(reference "C1")
@@
 		)
 		(instances
-			(project "Yuzu"
+			(project "yuzu-pcb"
 				(path "/170d21ec-bdb4-4292-838e-4735dd755299"
 					(reference "#PWR06")
@@
 			)
 		)
-		(property "Footprint" "yuzu:E73-2G4M08S1C-52840_SMD"
+		(property "Footprint" "yuzu:E73(2G4M08S1C) JLCPCB"
 			(at 85.09 130.81 0)
 			(effects
@@
 		)
 		(instances
-			(project "Yuzu"
+			(project "yuzu-pcb"
 				(path "/170d21ec-bdb4-4292-838e-4735dd755299"
 					(reference "U1")
@@
 			)
 		)
-		(property "Footprint" "Capacitor_SMD:C_0402_1005Metric_Pad0.74x0.62mm_HandSolder"
+		(property "Footprint" "Capacitor_SMD:C_0402_1005Metric"
 			(at 30.48 134.3152 0)
 			(effects
@@
 		)
 		(instances
-			(project "Yuzu"
+			(project "yuzu-pcb"
 				(path "/170d21ec-bdb4-4292-838e-4735dd755299"
 					(reference "C3")

Commit message: Updated schematic and pcb
Parts:
- added D2: White, LED_SMD:LED_0603_1608Metric, symbol Device:LED
- added J2: Conn_01x04, Connector_JST:JST_SH_BM04B-SRSS-TB_1x04-1MP_P1.00mm_Vertical, symbol Connector_Generic:Conn_01x04
- added R4: 1K, Resistor_SMD:R_0603_1608Metric, symbol Device:R
- added TP1: A1, yuzu:TestPoint_THTPad, symbol Connector:TestPoint
- added TP10: VD, yuzu:TestPoint_THTPad, symbol Connector:TestPoint
- added TP2: A4, yuzu:TestPoint_THTPad, symbol Connector:TestPoint
- added TP3: A0, yuzu:TestPoint_THTPad, symbol Connector:TestPoint
- added TP4: A5, yuzu:TestPoint_THTPad, symbol Connector:TestPoint
- added TP5: GD, yuzu:TestPoint_THTPad, symbol Connector:TestPoint
- added TP6: CL, yuzu:TestPoint_THTPad, symbol Connector:TestPoint
- added TP7: IO, yuzu:TestPoint_THTPad, symbol Connector:TestPoint
- added TP8: WO, yuzu:TestPoint_THTPad, symbol Connector:TestPoint
- added TP9: RS, yuzu:TestPoint_THTPad, symbol Connector:TestPoint
- BT1: footprint Battery:BatteryHolder_Keystone_3034_1x20mm -> Battery:BatteryHolder_Keystone_1060_1x2032
- J1: now left out of the parts list
- SW1: footprint Button_Switch_SMD:SW_SPST_B3U-1000P -> yuzu:RKB2SJG250SMTRLFS; symbol Switch:SW_SPST -> Switch:SW_DPST; LCSC (none) -> C2927788
- U1: footprint yuzu:E73(2G4M08S1C) JLCPCB -> yuzu:E73(2G4M08S1C) JLCPCB_2
Connections:
- net GND: now also SW1.3, J2.1 (Pin_1), R4.2, TP5.1
- net RED_LED: now also U1.9 (P0.31/AIN7); no longer U1.6 (P1.13)
- net RESET: now also SW1.4, TP9.1
- net SCL: now also U1.15 (P0.05/AIN3), J2.4 (Pin_4); no longer U1.17 (P1.09)
- net SDA: now also U1.17 (P1.09), J2.3 (Pin_3); no longer U1.15 (P0.05/AIN3)
- net SWCLK: now also TP6.1
- net SWDIO: now also TP7.1
- net SWO: now also TP8.1
- net nrf_VDD: now also J2.2 (Pin_2), TP10.1
- net XL2: now reaches C3.1, U1.13 (P0.01/XL2), X2.1
- net XL1: now reaches C1.1, U1.11 (P0.00/XL1), X2.2
- net WHITE_LED: now reaches U1.10 (P0.30/AIN6)
- net WHITE_LED: now also D2.2 (A)
- net at U1.3 (P0.03/AIN1): now also TP1.1
- net at U1.4 (P0.28/AIN4): now also TP2.1
- net at U1.7 (P0.02/AIN0): now also TP3.1
- net at U1.8 (P0.29/AIN5): now also TP4.1
- new net: D2.1 (K), R4.1
- no-connect marks 30 -> 23
Other:
- note added: "TODO: graphics?"
- note removed: "TODO: VDIV Decoupling capacitors? make sure can purchase connectors"
- moved on the sheet: C1, C3, D1, J1, R1, U1, X2

Commit message: Sent for production
Connections:
- net GND: now also SW1.2; no longer SW1.3
- net RESET: now also SW1.3; no longer SW1.2
